File: Routage.sch (KiCad schematic (older format))
At the start: 52 parts, among them J2 Conn_01x02, J3 Conn_01x03, Q1 2N2907, Q10 TIP32, Q11 BD138, Q12 TIP31, Q13 2N2222, Q2 2N2907, Q3 2N2907, Q4 2N2222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

Commit message: ERC (pb GND, 12V et TNjack) + attribution des empreintres (pb C10u, incertitude R11 & R12 => 2W , Rpot?)
Parts:
- C1, C3: footprint (none) -> CmpAmpliAudio:CP_Radial_D8.0mm_P5.00mm
- C10, C8: footprint (none) -> CmpAmpliAudio:CP_Radial_D12.5mm_P5.00mm
- C11, C2, C5, C7, C9: footprint (none) -> CmpAmpliAudio:C_Rect_L7.2mm_W3.5mm_P5.00mm_FKS2_FKP2_MKS2_MKP2
- D1, D2: footprint (none) -> CmpAmpliAudio:D_DO-35_SOD27_P10.16mm_Horizontal
- Dz1: footprint Diode_SMD:D_SOD-323 -> CmpAmpliAudio:D_DO-35_SOD27_P10.16mm_Horizontal
- HS1, HS2: footprint (none) -> CmpAmpliAudio:Heatsink_Fischer_SK104-STC-STIC_35x13mm_2xDrill2.5mm
- J2: footprint (none) -> CmpAmpliAudio:PhoenixContact_MSTBVA_2,5_2-G-5,08_1x02_P5.08mm_Vertical
- J3: footprint (none) -> CmpAmpliAudio:PhoenixContact_MSTBVA_2,5_3-G-5,08_1x03_P5.08mm_Vertical
- Q1, Q13, Q2, Q3, Q4, Q5, Q6, Q7: footprint (none) -> CmpAmpliAudio:TO-18-3
- Q10, Q12: footprint (none) -> CmpAmpliAudio:TO-220-3_Vertical
- Q11, Q8, Q9: footprint (none) -> CmpAmpliAudio:TO-126-3_Vertical
- R1, R10, R13, R14, R15, R16, R17, R2, R3, R4, R5, R6, R7, R8, R9: footprint (none) -> CmpAmpliAudio:R_Axial_DIN0207_L6.3mm_D2.5mm_P10.16mm_Horizontal
- R11, R12: footprint (none) -> CmpAmpliAudio:R_Axial_DIN0516_L15.5mm_D5.0mm_P20.32mm_Horizontal
- U1: renamed from U?; footprint (none) -> Mes_Empreintes:Relais_OJ-SS-112LMH2,005
- U2: footprint (none) -> CmpAmpliAudio:Jack_35RAPC2AV

Commit message: Version 1 du placement avec changement de librairie fait
Parts:
- C4, C6: footprint (none) -> CmpAmpliAudio:CP_Radial_D8.0mm_P5.00mm
- RV1, RV2: footprint (none) -> CmpAmpliAudio:Potentiometer_Bourns_3296W_Vertical
- U2: symbol CmpAmpliAudio:Jack_Mono -> Routage-rescue:Jack_Mono-CmpAmpliAudio
Changed lines of the file:
@@
 encoding utf-8
 Sheet 1 1
-Title ""
-Date ""
-Rev ""
-Comp ""
+Title "Routage BE_Elec"
+Date "2021-04-01"
+Rev "V0"
+Comp "GEI INSA"
 Comment1 ""
 Comment2 ""
@@
 F 0 "RV2" H 4030 2846 50  0000 R CNN
 F 1 "R_POT" H 4030 2755 50  0000 R CNN
-F 2 "" H 4100 2800 50  0001 C CNN
+F 2 "CmpAmpliAudio:Potentiometer_Bourns_3296W_Vertical" H 4100 2800 50  0001 C CNN
 F 3 "~" H 4100 2800 50  0001 C CNN
 	1    4100 2800
@@
 F 0 "RV1" H 4581 2546 50  0000 R CNN
 F 1 "R_POT" H 4581 2455 50  0000 R CNN
-F 2 "" H 4650 2500 50  0001 C CNN
+F 2 "CmpAmpliAudio:Potentiometer_Bourns_3296W_Vertical" H 4650 2500 50  0001 C CNN
 F 3 "~" H 4650 2500 50  0001 C CNN
 	1    4650 2500
@@
 	8700 5050 8700 5200
 $Comp
-L CmpAmpliAudio:Jack_Mono U2
+L Routage-rescue:Jack_Mono-CmpAmpliAudio U2
 U 1 1 6059FCE6
 P 1250 3300
@@
 F 0 "C4" H 2218 6296 50  0000 L CNN
 F 1 "10u" H 2218 6205 50  0000 L CNN
-F 2 "" H 2138 6100 50  0001 C CNN
+F 2 "CmpAmpliAudio:CP_Radial_D8.0mm_P5.00mm" H 2138 6100 50  0001 C CNN
 F 3 "~" H 2100 6250 50  0001 C CNN
 	1    2100 6250
@@
 F 0 "C6" H 2218 6846 50  0000 L CNN
 F 1 "10u" H 2218 6755 50  0000 L CNN
-F 2 "" H 2138 6650 50  0001 C CNN
+F 2 "CmpAmpliAudio:CP_Radial_D8.0mm_P5.00mm" H 2138 6650 50  0001 C CNN
 F 3 "~" H 2100 6800 50  0001 C CNN
 	1    2100 6800

Commit message: V1 du routage + Changement placement + rajout diode + Pb masse
Parts:
- added D3, D4: 1N4001, Diode_THT:D_DO-41_SOD81_P10.16mm_Horizontal, symbol Diode:1N4001
Connections:
- net +12V: now also D3.1 (K)
- net -12V: now also D4.2 (A)
- net GND: now also D3.2 (A), D4.1 (K)
Changed lines of the file:
@@
 	2100 6000 2100 6100
-Wire Wire Line
-	2100 6950 2100 7100
 Wire Wire Line
 	2100 7100 1600 7100
@@
 	2100 6500 2100 6650
 Wire Wire Line
-	2100 6500 2650 6500
+	2100 6500 2450 6500
 $Comp
 L Relay:Relay_1CT U1
@@
 L power:GND #PWR0101
 U 1 1 606B7903
-P 2650 6650
-F 0 "#PWR0101" H 2650 6400 50  0001 C CNN
-F 1 "GND" H 2655 6477 50  0000 C CNN
-F 2 "" H 2650 6650 50  0001 C CNN
-F 3 "" H 2650 6650 50  0001 C CNN
-	1    2650 6650
+P 2900 6650
+F 0 "#PWR0101" H 2900 6400 50  0001 C CNN
+F 1 "GND" H 2905 6477 50  0000 C CNN
+F 2 "" H 2900 6650 50  0001 C CNN
+F 3 "" H 2900 6650 50  0001 C CNN
+	1    2900 6650
 	1    0    0    -1
 $EndComp
 Wire Wire Line
-	2650 6500 2650 6650
+	2900 6500 2900 6650
 $Comp
 L power:GND #PWR0102
@@
 Wire Wire Line
 	1950 3850 1950 4150
+$Comp
+L Diode:1N4001 D3
+U 1 1 6073897A
+P 2450 6250
+F 0 "D3" V 2404 6330 50  0000 L CNN
+F 1 "1N4001" V 2495 6330 50  0000 L CNN
+F 2 "Diode_THT:D_DO-41_SOD81_P10.16mm_Horizontal" H 2450 6075 50  0001 C CNN
+F 3 "http://www.vishay.com/docs/88503/1n4001.pdf" H 2450 6250 50  0001 C CNN
+	1    2450 6250
+	0    1    1    0
+$EndComp
+$Comp
+L Diode:1N4001 D4
+U 1 1 60738FEF
+P 2450 6800
+F 0 "D4" V 2404 6880 50  0000 L CNN
+F 1 "1N4001" V 2495 6880 50  0000 L CNN
+F 2 "Diode_THT:D_DO-41_SOD81_P10.16mm_Horizontal" H 2450 6625 50  0001 C CNN
+F 3 "http://www.vishay.com/docs/88503/1n4001.pdf" H 2450 6800 50  0001 C CNN
+	1    2450 6800
+	0    1    1    0
+$EndComp
+Wire Wire Line
+	2450 6500 2450 6400
+Connection ~ 2450 6500
+Wire Wire Line
+	2450 6100 2450 6000
+Wire Wire Line
+	2450 6000 2100 6000
+Connection ~ 2100 6000
+Wire Wire Line
+	2450 6500 2450 6650
+Wire Wire Line
+	2100 6950 2100 7100
+Wire Wire Line
+	2100 7100 2450 7100
+Wire Wire Line
+	2450 7100 2450 6950
+Connection ~ 2100 7100
+Wire Wire Line
+	2450 6500 2900 6500
 $EndSCHEMATC
